File: hackboards/openboard/PCB/openboard.kicad_pcb (KiCad board)
At the start: 2 copper layers, 381.9 x 134.3 mm, 207 parts, among them U1 Raspberry_Pi_Pico

Commit message: did stuff
Connections:
- S100 pad 1: COL11 -> COL10
- S101 pad 1: COL12 -> COL11
- S102 pad 1: COL13 -> COL12
- S88 pad 1: COL13 -> COL12
- S94 pad 1: COL1 -> COL0
- S95 pad 1: COL2 -> COL1
- S96 pad 1: COL3 -> COL2
- S97 pad 1: COL6 -> COL5
- S99 pad 1: COL10 -> COL9
Routing:
- net COL0: track 424.1 -> 647.0 mm
- net COL13: track 339.5 -> 119.4 mm, vias 1 -> 0
- net COL4: track 349.2 -> 528.2 mm
- net COL5: track 343.6 -> 509.0 mm
- net COL2: track 434.3 -> 592.1 mm
- net COL1: track 456.7 -> 614.1 mm
- net COL6: track 354.2 -> 493.9 mm, vias 1 -> 0
- net COL3: track 409.5 -> 547.0 mm
- net COL8: track 290.2 -> 426.5 mm
- net COL7: track 324.7 -> 450.5 mm, vias 0 -> 1
- net COL10: track 276.2 -> 385.3 mm, vias 3 -> 1
- net COL11: track 397.4 -> 357.5 mm
- net COL12: track 364.0 -> 336.5 mm
- net COL18: track 139.9 -> 113.7 mm, vias 3 -> 1
- net COL9: track 433.0 -> 415.2 mm
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