File: hackboards/openboard/PCB/openboard.kicad_sch (KiCad schematic)
At the start: 201 parts, among them U1 Raspberry_Pi_Pico

Commit message: did stuff
Connections:
- net COL0: now also S94.1
- net COL1: now also S95.1; no longer S94.1
- net COL10: now also S100.1; no longer S99.1
- net COL11: now also S101.1; no longer S100.1
- net COL12: now also S102.1, S88.1; no longer S101.1
- net COL13: no longer S102.1, S88.1
- net COL2: now also S96.1; no longer S95.1
- net COL3: no longer S96.1
- net COL5: now also S97.1
- net COL6: no longer S97.1
- net COL9: now also S99.1
Other:
- moved on the sheet: D100, D101, D102, D88, D94, D95, D96, D97, D99, S100, S101, S102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
