File: hackboards/clearboard/PCB/clearboard.kicad_pcb (KiCad board)
At the start: 2 copper layers, 381.9 x 134.3 mm, 207 parts, among them U1 Raspberry_Pi_Pico

Commit message: I think I finalized my pcb
Routing:
- net COL2: track 592.1 -> 585.0 mm
- removed copper zone on F.Cu, net (none)
